File: Kicad_Projet/Shield/Shield.kicad_pcb (KiCad board)
At the start: 2 copper layers, 68.6 x 53.3 mm, 25 parts, among them J1 Power, J2 Digital/PWM, J3 Analog, J4 Digital/PWM, U2 LTC1050

Commit message: connectique
Parts:
- removed C3: 100n, Capacitor_THT:C_Disc_D4.3mm_W1.9mm_P5.00mm
- added C6: 100n, Capacitor_THT:C_Disc_D4.3mm_W1.9mm_P5.00mm, F.Cu at (163.0, 60.0)
- R6: value 10k -> 47k
- moved U1 85.8 mm to (162.0, 80.0), turned to 90 degrees
- moved Encodeur1 78.7 mm to (157.5, 58.5)
- moved R6 45.4 mm to (157.0, 92.6), turned to 90 degrees
- moved C4 39.8 mm to (122.9, 93.5), turned to 180 degrees
- moved U2 38.0 mm to (118.7, 76.5)
- moved R2 35.9 mm to (114.4, 94.2)
- moved Flex_Sensor1 32.7 mm to (151.5, 85.0), turned to 90 degrees
- moved Potentiometre1 32.7 mm to (129.0, 57.0), turned to -90 degrees
- moved C1 27.7 mm to (118.4, 89.0)
- moved Bluetooth1 25.6 mm to (147.5, 62.3), turned to -90 degrees
- moved R1 21.0 mm to (132.6, 88.5), turned to 180 degrees
- moved Capteur_Graphite1 19.7 mm to (126.7, 80.5)
- moved C2 17.4 mm to (138.5, 82.5), turned to 180 degrees
- moved R4 16.7 mm to (141.8, 77.3), turned to 180 degrees
- moved R5 15.9 mm to (136.9, 93.5), turned to 180 degrees
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Connections:
- C1 pad 1: R3 -> Net-(U2-+)
- R1 pad 2: R3 -> Net-(U2-+)
- R2 pad 1: R3 -> Net-(U2-+)
- U2 pad 3: R3 -> Net-(U2-+)
Routing:
- net ADC: track 0.00 -> 29.5 mm
- net Net-(U2-+): track 0.00 -> 23.7 mm
- net Net-(C2-Pad1): track 0.00 -> 18.2 mm
- net +5V: track 0.00 -> 12.1 mm
- net Net-(Capteur_Graphite1-SCRC): track 0.00 -> 9.13 mm
- net R3: track 0.00 -> 6.19 mm
- added copper zone on B.Cu, net GND
Other:
- board text added: "Aliénor Jarry Bastien Maïs"
