File: Kicad_Projet/Shield/Shield.kicad_sch (KiCad schematic)
At the start: 21 parts, among them J1 Power, J2 Digital/PWM, J3 Analog, J4 Digital/PWM, U2 LTC1050

Commit message: connectique
Parts:
- removed C3: 100n, Capacitor_THT:C_Disc_D4.3mm_W1.9mm_P5.00mm, symbol Device:C
- added C6: 100n, Capacitor_THT:C_Disc_D4.3mm_W1.9mm_P5.00mm, symbol Device:C
- R6: value 10k -> 47k
Connections:
- net CLK: now also C6.2
- net GND: now also C6.1
- net R3: no longer C1.1, R1.2, R2.1, U2.3 (+)
- new net: C1.1, R1.2, R2.1, U2.3 (+)

Commit message: pcb and mask
Connections:
- net +5V: now also Potentiometre1.8 (VDD)
- net GND: now also Potentiometre1.4 (VSS)
- net A4 renamed SDA
- no-connect marks 14 -> 12
Changed lines of the file:
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@@
 	)
 	(no_connect
-		(at 31.75 167.64)
-	)
-	(no_connect
 		(at 26.67 36.83)
 	)
@@
 	)
 	(no_connect
-		(at 54.61 156.21)
-	)
-	(no_connect
 		(at 82.55 31.75)
 	)
@@
 	(wire
 		(pts
-			(xy 167.64 73.66) (xy 167.64 50.8)
+			(xy 167.64 73.66) (xy 167.64 64.77)
 		)
 		(stroke
@@
 	(wire
 		(pts
-			(xy 222.25 43.18) (xy 229.87 43.18)
-		)
-		(stroke
-			(width 0)
-			(type default)
-		)
-	)
-	(wire
-		(pts
 			(xy 27.94 130.81) (xy 27.94 127)
 		)
@@
 	(wire
 		(pts
-			(xy 250.19 80.01) (xy 250.19 88.9)
+			(xy 54.61 156.21) (xy 59.69 156.21)
 		)
 		(stroke
@@
 	(wire
 		(pts
-			(xy 222.25 43.18) (xy 222.25 67.31)
+			(xy 250.19 80.01) (xy 250.19 88.9)
 		)
 		(stroke
@@
 	(wire
 		(pts
+			(xy 222.25 60.96) (xy 222.25 67.31)
+		)
+		(stroke
+			(width 0)
+			(type default)
+		)
+	)
+	(wire
+		(pts
 			(xy 240.03 80.01) (xy 250.19 80.01)
 		)
@@
 	(wire
 		(pts
-			(xy 229.87 43.18) (xy 229.87 41.91)
-		)
-		(stroke
-			(width 0)
-			(type default)
-		)
-	)
-	(wire
-		(pts
 			(xy 69.85 29.21) (xy 82.55 29.21)
 		)
@@
 	(wire
 		(pts
+			(xy 27.94 167.64) (xy 31.75 167.64)
+		)
+		(stroke
+			(width 0)
+			(type default)
+		)
+	)
+	(wire
+		(pts
 			(xy 69.85 74.93) (xy 82.55 74.93)
 		)
@@
 		)
 	)
-	(global_label "A4"
-		(shape input)
-		(at 87.63 162.56 180)
-		(fields_autoplaced yes)
-		(effects
-			(font
-				(size 1.27 1.27)
-			)
-			(justify right)
-		)
-		(property "Intersheetrefs" "${INTERSHEET_REFS}"
-			(at 82.2516 162.56 0)
-			(effects
-				(font
-					(size 1.27 1.27)
-				)
-				(justify right)
-				(hide yes)
-			)
-		)
-	)
 	(global_label "CS"
 		(shape input)
@@
 		)
 	)
+	(global_label "SCL"
+		(shape input)
+		(at 82.55 26.67 0)
+		(fields_autoplaced yes)
+		(effects
+			(font
+				(size 1.27 1.27)
+			)
+			(justify left)
+		)
+		(property "Intersheetrefs" "${INTERSHEET_REFS}"
+			(at 89.1379 26.67 0)
+			(effects
+				(font
+					(size 1.27 1.27)
+				)
+				(justify left)
+				(hide yes)
+			)
+		)
+	)
 	(global_label "TXD"
 		(shape input)
@@
 		)
 	)
+	(global_label "SDA"
+		(shape input)
+		(at 29.21 69.85 180)
+		(fields_autoplaced yes)
+		(effects
+			(font
+				(size 1.27 1.27)
+			)
+			(justify right)
+		)
+		(property "Intersheetrefs" "${INTERSHEET_REFS}"
+			(at 22.5616 69.85 0)
+			(effects
+				(font
+					(size 1.27 1.27)
+				)
+				(justify right)
+				(hide yes)
+			)
+		)
+	)
+	(global_label "SDA"
+		(shape input)
+		(at 82.55 29.21 0)
+		(fields_autoplaced yes)
+		(effects
+			(font
+				(size 1.27 1.27)
+			)
+			(justify left)
+		)
+		(property "Intersheetrefs" "${INTERSHEET_REFS}"
+			(at 89.1984 29.21 0)
+			(effects
+				(font
+					(size 1.27 1.27)
+				)
+				(justify left)
+				(hide yes)
+			)
+		)
+	)
 	(global_label "SCL"
 		(shape input)
@@
 		)
 	)
+	(global_label "SDA"
+		(shape input)
+		(at 87.63 162.56 180)
+		(fields_autoplaced yes)
+		(effects
+			(font
+				(size 1.27 1.27)
+			)
+			(justify right)
+		)
+		(property "Intersheetrefs" "${INTERSHEET_REFS}"
+			(at 80.9816 162.56 0)
+			(effects
+				(font
+					(size 1.27 1.27)
+				)
+				(justify right)
+				(hide yes)
+			)
+		)
+	)
 	(global_label "SW"
 		(shape input)
@@
 		)
 	)
-	(global_label "A4"
-		(shape input)
-		(at 29.21 69.85 180)
-		(fields_autoplaced yes)
-		(effects
-			(font
-				(size 1.27 1.27)
-			)
-			(justify right)
-		)
-		(property "Intersheetrefs" "${INTERSHEET_REFS}"
-			(at 23.8316 69.85 0)
-			(effects
-				(font
-					(size 1.27 1.27)
-				)
-				(justify right)
-				(hide yes)
-			)
-		)
-	)
 	(symbol
 		(lib_id "Connector_Generic:Conn_01x08")
@@
 	)
 	(symbol
+		(lib_id "power:+5V")
+		(at 59.69 156.21 270)
+		(unit 1)
+		(exclude_from_sim no)
+		(in_bom yes)
+		(on_board yes)
+		(dnp no)
+		(fields_autoplaced yes)
+		(property "Reference" "#PWR028"
+			(at 55.88 156.21 0)
+			(effects
+				(font
+					(size 1.27 1.27)
+				)
+				(hide yes)
+			)
+		)
+		(property "Value" "+5V"
+			(at 63.5 156.2099 90)
+			(effects
+				(font
+					(size 1.27 1.27)
+				)
+				(justify left)
+			)
+		)
+		(property "Footprint" ""
+			(at 59.69 156.21 0)
+			(effects
+				(font
+					(size 1.27 1.27)
+				)
+				(hide yes)
+			)
+		)
+		(property "Datasheet" ""
+			(at 59.69 156.21 0)
+			(effects
+				(font
+					(size 1.27 1.27)
+				)
+				(hide yes)
+			)
+		)
+		(property "Description" "Power symbol creates a global label with name \"+5V\""
+			(at 59.69 156.21 0)
+			(effects
+				(font
+					(size 1.27 1.27)
+				)
+				(hide yes)
+			)
+		)
+		(pin "1"
+		)
+		(instances
+			(project "Shield"
+				(path "/e63e39d7-6ac0-4ffd-8aa3-1841a4541b55"
+					(reference "#PWR028")
+					(unit 1)
+				)
+			)
+		)
+	)
+	(symbol
 		(lib_id "ma_librairie:Servo_moteur")
 		(at 162.56 120.65 0)
@@
 	(symbol
 		(lib_id "power:GND")
+		(at 27.94 167.64 0)
+		(unit 1)
+		(exclude_from_sim no)
+		(in_bom yes)
+		(on_board yes)
+		(dnp no)
+		(fields_autoplaced yes)
+		(property "Reference" "#PWR027"
+			(at 27.94 173.99 0)
+			(effects
+				(font
+					(size 1.27 1.27)
+				)
+				(hide yes)
+			)
+		)
+		(property "Value" "GND"
+			(at 27.94 172.72 0)
+			(effects
+				(font
+					(size 1.27 1.27)
+				)
+			)
+		)
+		(property "Footprint" ""
+			(at 27.94 167.64 0)
+			(effects
+				(font
+					(size 1.27 1.27)
+				)
+				(hide yes)
+			)
+		)
+		(property "Datasheet" ""
+			(at 27.94 167.64 0)
+			(effects
+				(font
+					(size 1.27 1.27)
+				)
+				(hide yes)
+			)
+		)
+		(property "Description" "Power symbol creates a global label with name \"GND\" , ground"
+			(at 27.94 167.64 0)
+			(effects
+				(font
+					(size 1.27 1.27)
+				)
+				(hide yes)
+			)
+		)
+		(pin "1"
+		)
+		(instances
+			(project "Shield"
+				(path "/e63e39d7-6ac0-4ffd-8aa3-1841a4541b55"
+					(reference "#PWR027")
+					(unit 1)
+				)
+			)
+		)
+	)
+	(symbol
+		(lib_id "power:GND")
 		(at 205.74 92.71 0)
 		(unit 1)
@@
 	(symbol
 		(lib_id "power:+5V")
-		(at 229.87 41.91 0)
+		(at 222.25 60.96 0)
 		(unit 1)
 		(exclude_from_sim no)
@@
 		(fields_autoplaced yes)
 		(property "Reference" "#PWR09"
-			(at 229.87 45.72 0)
+			(at 222.25 64.77 0)
 			(effects
 				(font
@@
 		)
 		(property "Value" "+5V"
-			(at 229.87 36.83 0)
+			(at 222.25 55.88 0)
 			(effects
 				(font
@@
 		)
 		(property "Footprint" ""
-			(at 229.87 41.91 0)
+			(at 222.25 60.96 0)
 			(effects
 				(font
@@
 		)
 		(property "Datasheet" ""
-			(at 229.87 41.91 0)
+			(at 222.25 60.96 0)
 			(effects
 				(font
@@
 		)
 		(property "Description" "Power symbol creates a global label with name \"+5V\""
-			(at 229.87 41.91 0)
+			(at 222.25 60.96 0)
 			(effects
 				(font
@@
 	(symbol
 		(lib_id "power:+5V")
-		(at 167.64 50.8 0)
+		(at 167.64 64.77 0)
 		(unit 1)
 		(exclude_from_sim no)
@@
 		(fields_autoplaced yes)
 		(property "Reference" "#PWR015"
-			(at 167.64 54.61 0)
+			(at 167.64 68.58 0)
 			(effects
 				(font
@@
 		)
 		(property "Value" "+5V"
-			(at 167.64 45.72 0)
+			(at 167.64 59.69 0)
 			(effects
 				(font
@@
 		)
 		(property "Footprint" ""
-			(at 167.64 50.8 0)
+			(at 167.64 64.77 0)
 			(effects
 				(font
@@
 		)
 		(property "Datasheet" ""
-			(at 167.64 50.8 0)
+			(at 167.64 64.77 0)
 			(effects
 				(font
@@
 		)
 		(property "Description" "Power symbol creates a global label with name \"+5V\""
-			(at 167.64 50.8 0)
+			(at 167.64 64.77 0)
 			(effects
 				(font
